Commit message: changed rviz file and parameters in macro

File: urdf/assembled_macro.xacro (robot description, xacro)
@@ -25,5 +25,5 @@
                     <box size="${length} ${width} ${height}"/>
                 </geometry>
-                <origin rpy="0 0 0" xyz="0 0 ${height / 2}"/>
+                <origin rpy="0 0 0" xyz="0 0 -${height}"/>
             </visual>
             <collision>
@@ -31,5 +31,5 @@
                     <box size="${length} ${width} ${height}"/>
                 </geometry>
-                <origin rpy="0 0 0" xyz="0 0 ${height / 2}"/>
+                <origin rpy="0 0 0" xyz="0 0 -${height}"/>
             </collision>
         </link>

Commit message: fixed world and table frames

File: urdf/assembled_macro.xacro (robot description, xacro)
@@ -5,4 +5,7 @@
     <xacro:property name="width" value="0.5"/>
     <xacro:property name="height" value="0.5"/>
+    <material name="blue">
+        <color rgba="0 0 0.8 0.5"/>
+    </material>
     <xacro:macro name="assembled_robot" params="
         parent
@@ -16,7 +19,7 @@
         <!--  this joint fixes the table to the world link given as a parameter -->
         <joint name="table_base_joint" type="fixed">
-            <xacro:insert_block name="origin"/>
             <parent link="${parent}"/>
             <child link="table"/>
+            <origin xyz="0 0 ${height}" rpy="0 0 0"/>
         </joint>
         <link name="table">
@@ -25,5 +28,6 @@
                     <box size="${length} ${width} ${height}"/>
                 </geometry>
-                <origin rpy="0 0 0" xyz="0 0 -${height}"/>
+                <origin rpy="0 0 0" xyz="0 0 -${height/2}"/>
+                <material name="blue"/>
             </visual>
             <collision>
@@ -31,5 +35,5 @@
                     <box size="${length} ${width} ${height}"/>
                 </geometry>
-                <origin rpy="0 0 0" xyz="0 0 -${height}"/>
+                <origin rpy="0 0 0" xyz="0 0 -${height/2}"/>
             </collision>
         </link>

Commit message: changed orientaton of robot

File: urdf/assembled_macro.xacro (robot description, xacro)
@@ -2,8 +2,8 @@
 <robot xmlns:xacro="http://ros.org/wiki/xacro">
     <xacro:include filename="$(find ur_description)/urdf/ur_macro.xacro"/>
-    <xacro:property name="length" value="0.5"/>
-    <xacro:property name="width" value="0.5"/>
-    <xacro:property name="height" value="0.5"/>
-    <material name="blue">
+    <xacro:property name="length" value="0.60"/>
+    <xacro:property name="width" value="0.75"/>
+    <xacro:property name="height" value="0.90"/>
+    <material name="blue_table">
         <color rgba="0 0 0.8 0.5"/>
     </material>
@@ -21,5 +21,5 @@
             <parent link="${parent}"/>
             <child link="table"/>
-            <origin xyz="0 0 ${height}" rpy="0 0 0"/>
+            <origin xyz="0 0 ${height}" rpy="0 0 -${pi/4}"/>
         </joint>
         <link name="table">
@@ -28,6 +28,6 @@
                     <box size="${length} ${width} ${height}"/>
                 </geometry>
-                <origin rpy="0 0 0" xyz="0 0 -${height/2}"/>
-                <material name="blue"/>
+                <origin xyz="0 0 -${height/2}" rpy="0 0 ${pi/4}" />
+                <material name="blue_table"/>
             </visual>
             <collision>
@@ -35,5 +35,5 @@
                     <box size="${length} ${width} ${height}"/>
                 </geometry>
-                <origin rpy="0 0 0" xyz="0 0 -${height/2}"/>
+                <origin xyz="0 0 -${height/2}" rpy="0 0 ${pi/4}" />
             </collision>
         </link>
@@ -42,5 +42,5 @@
             <parent link="table"/>
             <child link="robot_mount"/>
-            <origin xyz="0 0 0" rpy="0 0 ${pi}"/>
+            <origin xyz="0 0 0" rpy="0 0 0"/>
         </joint>
         <!-- This will create the specific robot -->
@@ -48,5 +48,5 @@
             name="${ur_type}"
             tf_prefix="${ur_type}_"
-            parent="robot_mount"
+            parent="${parent}"
             joint_limits_parameters_file="${joint_limits_parameters_file}"
             kinematics_parameters_file="${kinematics_parameters_file}"
@@ -54,5 +54,5 @@
             visual_parameters_file="${visual_parameters_file}"
         >
-            <origin xyz="0 0 0" rpy="0 0 0"/>
+            <origin xyz="0 0 ${height}" rpy="0 0 ${pi}"/>
         </xacro:ur_robot>
     </xacro:macro>

File: urdf/ur10_assembly.urdf.xacro (robot description, xacro)
@@ -18,5 +18,5 @@
         visual_parameters_file="$(arg visual_parameters_file)"
         >
-            <origin xyz="0 0 1" rpy="0 0 0"/>
+            <origin xyz="0 0 0" rpy="0 0 0"/>
     </xacro:assembled_robot>
 </robot>

Commit message: robotiq gripper added

File: urdf/assembled_macro.xacro (robot description, xacro)
@@ -2,9 +2,10 @@
 <robot xmlns:xacro="http://ros.org/wiki/xacro">
     <xacro:include filename="$(find ur_description)/urdf/ur_macro.xacro"/>
+    <xacro:include filename="$(find robotiq_description)/urdf/robotiq_2f_85_macro.urdf.xacro"/>
     <xacro:property name="length" value="0.60"/>
     <xacro:property name="width" value="0.75"/>
     <xacro:property name="height" value="0.90"/>
     <material name="blue_table">
-        <color rgba="0 0 0.8 0.5"/>
+        <color rgba="0 0 0.8 1"/>
     </material>
     <xacro:macro name="assembled_robot" params="
@@ -56,4 +57,12 @@
             <origin xyz="0 0 ${height}" rpy="0 0 ${pi}"/>
         </xacro:ur_robot>
+        <!-- This will create gripper -->
+        <xacro:robotiq_gripper
+            name="RobotiqGripper"
+            prefix="${ur_type}_"
+            parent="${ur_type}_flange"
+        >
+            <origin xyz="0 0 0" rpy="0 ${pi/2} 0"/>
+    </xacro:robotiq_gripper>
     </xacro:macro>
 </robot>

Commit message: tool macro added

File: urdf/assembled_macro.xacro (robot description, xacro)
@@ -3,4 +3,5 @@
     <xacro:include filename="$(find ur_description)/urdf/ur_macro.xacro"/>
     <xacro:include filename="$(find robotiq_description)/urdf/robotiq_2f_85_macro.urdf.xacro"/>
+    <xacro:include filename="$(find ur10_assembly)/urdf/tool_macro.xacro"/>
     <xacro:property name="length" value="0.60"/>
     <xacro:property name="width" value="0.75"/>
@@ -9,4 +10,5 @@
         <color rgba="0 0 0.8 1"/>
     </material>
+    <xacro:property name="gripper_name" value="robotiq_85"/>
     <xacro:macro name="assembled_robot" params="
         parent
@@ -64,5 +66,12 @@
         >
             <origin xyz="0 0 0" rpy="0 ${pi/2} 0"/>
-    </xacro:robotiq_gripper>
+        </xacro:robotiq_gripper>
+        <!-- This will create tool -->
+        <xacro:tool
+            name="tool"
+            prefix="${ur_type}_"
+            parent="${ur_type}_${gripper_name}_base_link"
+        >
+        </xacro:tool>
     </xacro:macro>
 </robot>
