Commit message: tool size changed to 0.17

File: urdf/tool_macro.xacro (robot description, xacro)
@@ -6,5 +6,5 @@
         parent">
         <xacro:property name="radius" value="0.01"/>
-        <xacro:property name="length" value="0.1"/>
+        <xacro:property name="length" value="0.17"/>
         <material name="red">
             <color rgba="0.8 0 0 1"/>

Commit message: meshes added for pointer

File: urdf/tool_macro.xacro (robot description, xacro)
@@ -19,5 +19,6 @@
             <visual>
                 <geometry>
-                    <cylinder radius="${radius}" length="${length}"/>
+                    <mesh filename="package://ur10_assembly/meshes/pointer.STL" scale="0.001 0.001 0.001"/>
+                    <!-- <cylinder radius="${radius}" length="${length}"/> -->
                 </geometry>
                 <material name="red"/>

Commit message: pointer modified with stl file

File: urdf/tool_macro.xacro (robot description, xacro)
@@ -5,6 +5,4 @@
         prefix
         parent">
-        <xacro:property name="radius" value="0.01"/>
-        <xacro:property name="length" value="0.17"/>
         <material name="red">
             <color rgba="0.8 0 0 1"/>
@@ -19,15 +17,19 @@
             <visual>
                 <geometry>
+                    <!-- Using scale in the mesh file because
+                        the STL file was created in millimeters
+                        and when imported in rviz, it thinks it is in meters.
+                        Therefore, scaling down the pointer.
+                    -->
                     <mesh filename="package://ur10_assembly/meshes/pointer.STL" scale="0.001 0.001 0.001"/>
-                    <!-- <cylinder radius="${radius}" length="${length}"/> -->
                 </geometry>
                 <material name="red"/>
-                <origin xyz="0 0 ${length/2}" rpy="0 0 0"/>
+                <origin xyz="0 0 0" rpy="0 0 0"/>
             </visual>
             <collision>
                 <geometry>
-                    <cylinder radius="${radius}" length="${length}"/>
+                    <mesh filename="package://ur10_assembly/meshes/pointer.STL" scale="0.001 0.001 0.001"/>
                 </geometry>
-                <origin xyz="0 0 ${length/2}"/>
+                <origin xyz="0 0 0"/>
             </collision>
             <xacro:default_inertial mass="0.5"/>
@@ -36,5 +38,5 @@
             <parent link="${parent}"/>
             <child link="${prefix}${name}"/>
-            <origin xyz="0 0 0.09" rpy="0 0 0"/>
+            <origin xyz="0 0 0.187" rpy="-${pi/2} 0 0"/>
         </joint>
     </xacro:macro>
